File: Hardware/CANIO/CANIO.kicad_sch (KiCad schematic)
At the start: 0 parts

Commit message: Fix names
Other:
- company: Kitsune Scientific -> Kitsune Robotics
Changed lines of the file:
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@@
     (title "CANIO")
     (rev "${REVISION}")
-    (company "Kitsune Scientific")
+    (company "Kitsune Robotics")
   )
   (sheet_instances

Commit message: Add kenwoodfox libs
Other:
- added sheet CANBUS (canbus.kicad_sch)
Changed lines of the file:
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@@
     (company "Kitsune Robotics")
+  )
+  (sheet (at 20.955 26.035) (size 29.845 35.56) (fields_autoplaced)
+    (stroke (width 0.1524) (type solid))
+    (fill (color 0 0 0 0.0000))
+    (property "Sheetname" "CANBUS" (at 20.955 25.3234 0)
+      (effects (font (size 1.27 1.27)) (justify left bottom))
+    )
+    (property "Sheetfile" "canbus.kicad_sch" (at 20.955 62.1796 0)
+      (effects (font (size 1.27 1.27)) (justify left top))
+    )
+    (instances
+      (project "CANIO"
+        (path "/894f620e-3404-4a40-a2a7-513bc1d5f99b" (page "2"))
+      )
+    )
   )
   (sheet_instances

Commit message: Add more boilerplate
Other:
- sheet CANBUS ports: added CLKOUT, CS, SCK, SI, SO; removed none
Changed lines of the file:
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@@
     (company "Kitsune Robotics")
   )
-  (sheet (at 20.955 26.035) (size 29.845 35.56) (fields_autoplaced)
+  (sheet (at 25.4 24.765) (size 12.7 41.91) (fields_autoplaced)
     (stroke (width 0.1524) (type solid))
     (fill (color 0 0 0 0.0000))
-    (property "Sheetname" "CANBUS" (at 20.955 25.3234 0)
+    (property "Sheetname" "CANBUS" (at 25.4 24.0534 0)
       (effects (font (size 1.27 1.27)) (justify left bottom))
     )
-    (property "Sheetfile" "canbus.kicad_sch" (at 20.955 62.1796 0)
+    (property "Sheetfile" "canbus.kicad_sch" (at 25.4 67.2596 0)
       (effects (font (size 1.27 1.27)) (justify left top))
     )
+    (pin "CLKOUT" output (at 38.1 64.77 0)
+      (effects (font (size 1.27 1.27)) (justify right))
+    )
+    (pin "SI" input (at 38.1 33.02 0)
+      (effects (font (size 1.27 1.27)) (justify right))
+    )
+    (pin "SO" output (at 38.1 31.115 0)
+      (effects (font (size 1.27 1.27)) (justify right))
+    )
+    (pin "CS" input (at 38.1 29.21 0)
+      (effects (font (size 1.27 1.27)) (justify right))
+    )
+    (pin "SCK" input (at 38.1 27.305 0)
+      (effects (font (size 1.27 1.27)) (justify right))
+    )
     (instances

Commit message: Add processor
Parts:
- added C101: 1u, Capacitor_SMD:C_0805_2012Metric, symbol Device:C_Small
- added C102, C104: 100nF, Capacitor_SMD:C_0805_2012Metric, symbol Device:C_Small
- added C103: 10uf, Capacitor_SMD:CP_Elec_4x3, symbol Device:C_Polarized_Small
- added C105: 1uF, Capacitor_SMD:C_0805_2012Metric, symbol Device:C_Small
- added D101: MBR0520LT, Diode_SMD:D_SOD-123, symbol Diode:MBR0520LT
- added D102: STAT, LED_SMD:LED_0805_2012Metric, symbol Device:LED
- added D103: PWR, LED_SMD:LED_0805_2012Metric, symbol Device:LED
- added J101: USBC, KenwoodFox:USB_C_Receptacle_XKB_U262-16XN-4BVC11_Full_Pads, symbol Connector:USB_C_Receptacle_USB2.0
- added J102: Tag Connect, Connector:Tag-Connect_TC2050-IDC-FP_2x05_P1.27mm_Vertical, symbol Connector_Generic:Conn_02x05_Odd_Even
- added R101, R102: 22R, Resistor_SMD:R_0805_2012Metric, symbol Device:R_Small
- added R103: 10k, Resistor_SMD:R_0805_2012Metric, symbol Device:R_Small
- added R104, R105: 5K1, Resistor_SMD:R_0805_2012Metric, symbol Device:R_Small
- added R106, R107: 1K, Resistor_SMD:R_0805_2012Metric, symbol Device:R_Small
- added U101: ATmega16U2, Package_QFP:TQFP-32_7x7mm_P0.8mm, symbol MCU_Microchip_ATmega:ATmega16U2-A
- added U102: LM1117MP-5.0, Package_TO_SOT_SMD:SOT-223-3_TabPin2, symbol Regulator_Linear:LM1117MP-5.0
Connections:
- new net: D101.2 (A), J101.A4 (VBUS), J101.A9 (VBUS), J101.B4 (VBUS), J101.B9 (VBUS)
- new net: J101.A5 (CC1), R105.2
- new net: J101.B5 (CC2), R104.2
- new net: R106.1, U101.6 (PD0)
- new net: D102.2 (A), R106.2
- new net: D103.2 (A), R107.2
- new net: C101.1, U101.27 (UCAP)
- new net: R101.2, U101.29 (D+)
- new net: R102.2, U101.30 (D-)
- new net +12V: C103.1, C104.1, U102.3 (VI)
- new net +5V: C102.1, C105.1, D101.1 (K), J102.2 (Pin_2), R103.2, R107.1, U101.31 (UVCC), U101.32 (AVCC), U101.4 (VCC), U102.2 (VO)
- new net CLKOUT: U101.1 (XTAL1)
- new net GND: C101.2, C102.2, C103.2, C104.2, C105.2, D102.1 (K), D103.1 (K), J101.A1 (GND), J101.A12 (GND), J101.B1 (GND), J101.B12 (GND), J101.S1 (SHIELD), J102.10 (Pin_10), R104.1, R105.1, U101.28 (UGND), U101.3 (GND), U102.1 (GND)
- new net ICSP_MISO: J102.9 (Pin_9), U101.17 (PB3)
- new net ICSP_MOSI: J102.1 (Pin_1), U101.16 (PB2)
- new net ICSP_RST: J102.5 (Pin_5), R103.1, U101.24 (PC1/~{RESET})
- new net ICSP_SCK: J102.7 (Pin_7), U101.15 (PB1)
- new net USB+: J101.A6 (D+), J101.B6 (D+), R101.1
- new net USB-: J101.A7 (D-), J101.B7 (D-), R102.1
- no-connect marks 0 -> 7
Other:
- note added: "Ask the Embed Discord about this! Weird to use the crystal output from another device!"
- note added: "USB"

Commit message: Bump
Changed lines of the file:
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@@
+    (stroke (width 0) (type default))
+  )
+  (wire (pts (xy 38.1 27.305) (xy 50.8 27.305))
     (stroke (width 0) (type default))
   )
@@
     (stroke (width 0) (type default))
   )
+  (wire (pts (xy 38.1 32.385) (xy 50.8 32.385))
+    (stroke (width 0) (type default))
+  )
   (wire (pts (xy 243.84 41.275) (xy 243.84 40.005))
     (stroke (width 0) (type default))
@@
   )
   (wire (pts (xy 20.32 179.705) (xy 29.845 179.705))
+    (stroke (width 0) (type default))
+  )
+  (wire (pts (xy 38.1 34.925) (xy 50.8 34.925))
     (stroke (width 0) (type default))
   )
@@
     (effects (font (size 1.27 1.27)) (justify right bottom))
   )
+  (label "ICSP_MOSI" (at 50.8 34.925 180) (fields_autoplaced)
+    (effects (font (size 1.27 1.27)) (justify right bottom))
+  )
   (label "ICSP_RST" (at 254.635 153.035 0) (fields_autoplaced)
     (effects (font (size 1.27 1.27)) (justify left bottom))
@@
   )
   (label "ICSP_SCK" (at 180.34 84.455 180) (fields_autoplaced)
+    (effects (font (size 1.27 1.27)) (justify right bottom))
+  )
+  (label "ICSP_SCK" (at 50.8 27.305 180) (fields_autoplaced)
+    (effects (font (size 1.27 1.27)) (justify right bottom))
+  )
+  (label "ICSP_MISO" (at 50.8 32.385 180) (fields_autoplaced)
     (effects (font (size 1.27 1.27)) (justify right bottom))
   )
@@
       (effects (font (size 1.27 1.27)) (justify right))
     )
-    (pin "SI" input (at 38.1 33.02 0)
+    (pin "SI" input (at 38.1 34.925 0)
       (effects (font (size 1.27 1.27)) (justify right))
     )
-    (pin "SO" output (at 38.1 31.115 0)
+    (pin "SO" output (at 38.1 32.385 0)
       (effects (font (size 1.27 1.27)) (justify right))
     )
-    (pin "CS" input (at 38.1 29.21 0)
+    (pin "CS" input (at 38.1 29.845 0)
       (effects (font (size 1.27 1.27)) (justify right))
     )

Commit message: Fix ERC
Parts:
- removed J101: USBC, KenwoodFox:USB_C_Receptacle_XKB_U262-16XN-4BVC11_Full_Pads, symbol Connector:USB_C_Receptacle_USB2.0
- added J103: PWR, Connector_JST:JST_XH_S2B-XH-A_1x02_P2.50mm_Horizontal, symbol Connector:Conn_01x02_Pin
- added P101: USB_C_Plug_USB2.0, KenwoodFox:USB_C_Receptacle_XKB_U262-16XN-4BVC11_Full_Pads, symbol Connector:USB_C_Plug_USB2.0
Connections:
- net +12V: now also J103.2 (Pin_2)
- net GND: now also J103.1 (Pin_1), P101.A1 (GND), P101.A12 (GND), P101.B1 (GND), P101.B12 (GND), P101.S1 (SHIELD)
- net USB+: now also P101.A6 (D+)
- net USB-: now also P101.A7 (D-)
- net at D101.2 (A): now also P101.A4 (VBUS), P101.A9 (VBUS), P101.B4 (VBUS), P101.B9 (VBUS)
- net at R105.2: now also P101.A5 (CC)
- net at R104.2: now also P101.B5 (VCONN)
- no-connect marks 7 -> 25
Other:
- sheet CANBUS ports: added INT, STBY; removed none
- note added: "Is standby pullup or down to standby?"

Commit message: Arthur is encouraging
Parts:
- removed C103: 10uf, Capacitor_SMD:CP_Elec_4x3, symbol Device:C_Polarized_Small
- removed C104: 100nF, Capacitor_SMD:C_0805_2012Metric, symbol Device:C_Small
- removed C105: 1uF, Capacitor_SMD:C_0805_2012Metric, symbol Device:C_Small
- removed D103: PWR, LED_SMD:LED_0805_2012Metric, symbol Device:LED
- removed R107: 1K, Resistor_SMD:R_0805_2012Metric, symbol Device:R_Small
- removed U102: LM1117MP-5.0, Package_TO_SOT_SMD:SOT-223-3_TabPin2, symbol Regulator_Linear:LM1117MP-5.0
Connections:
- net +12V is gone; now on net +5V: J103.2 (Pin_2)

Commit message: Always have a backup
Parts:
- added C103, C104: DNP, Capacitor_SMD:C_0603_1608Metric, symbol Device:C_Small
- added JP101: SolderJumper_2_Bridged, Jumper:SolderJumper-2_P1.3mm_Bridged2Bar_Pad1.0x1.5mm, symbol Jumper:SolderJumper_2_Bridged
- added Y101: DNP, Crystal:Crystal_SMD_3225-4Pin_3.2x2.5mm, symbol Device:Crystal_GND24
Connections:
- net CLKOUT: now also JP101.1 (A); no longer U101.1 (XTAL1)
- net GND: now also C103.2, C104.2, Y101.2, Y101.4
- net XTAL2: now reaches U101.2 (PC0/XTAL2)
- net XTAL2: now also C103.1, Y101.1
- new net XTAL1: C104.1, JP101.2 (B), U101.1 (XTAL1), Y101.3
- no-connect marks 25 -> 24
Other:
- note added: "16pf = (22pf)/2+5pf"
