File: Hardware/CANIO/CANIO.kicad_sch (KiCad schematic)
At the start: 18 parts, among them J102 Tag Connect, J103 PWR, P101 USB_C_Plug_USB2.0, U101 ATmega16U2, Y101 DNP

Commit message: My favorite switch
Parts:
- added R107: 10K, Resistor_SMD:R_0805_2012Metric, symbol Device:R_Small
- added SW101: RESET, Button_Switch_THT:SW_PUSH_6mm_H4.3mm, symbol Switch:SW_Push
Connections:
- net GND: now also R107.1, SW101.2
- net ICSP_RST: now also SW101.1
- net at U101.13 (~{HWB}/PD7): now also R107.2
- no-connect marks 24 -> 23
Changed lines of the file:
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@@
   (no_connect (at 50.8 29.845))
   (no_connect (at 278.765 153.035))
-  (no_connect (at 166.37 137.795))
   (no_connect (at 166.37 107.315))
   (no_connect (at 166.37 135.255))
@@
     (stroke (width 0) (type default))
   )
+  (wire (pts (xy 166.37 137.795) (xy 170.815 137.795))
+    (stroke (width 0) (type default))
+  )
   (wire (pts (xy 227.965 33.655) (xy 243.84 33.655))
     (stroke (width 0) (type default))
@@
     (stroke (width 0) (type default))
   )
+  (wire (pts (xy 255.27 130.175) (xy 266.7 130.175))
+    (stroke (width 0) (type default))
+  )
   (wire (pts (xy 227.965 31.115) (xy 254.635 31.115))
     (stroke (width 0) (type default))
@@
     (stroke (width 0) (type default))
   )
+  (wire (pts (xy 280.035 130.175) (xy 276.86 130.175))
+    (stroke (width 0) (type default))
+  )
   (wire (pts (xy 151.13 74.295) (xy 151.13 73.025))
     (stroke (width 0) (type default))
@@
     (stroke (width 0) (type default))
   )
+  (wire (pts (xy 178.435 137.795) (xy 175.895 137.795))
+    (stroke (width 0) (type default))
+  )
   (wire (pts (xy 146.05 73.025) (xy 148.59 73.025))
     (stroke (width 0) (type default))
@@
   )
   (wire (pts (xy 280.67 147.955) (xy 280.67 146.685))
+    (stroke (width 0) (type default))
+  )
+  (wire (pts (xy 280.035 132.08) (xy 280.035 130.175))
+    (stroke (width 0) (type default))
+  )
+  (wire (pts (xy 178.435 147.955) (xy 178.435 137.795))
     (stroke (width 0) (type default))
   )
@@
     (effects (font (size 1.27 1.27)) (justify right bottom))
   )
+  (label "ICSP_RST" (at 255.27 130.175 0) (fields_autoplaced)
+    (effects (font (size 1.27 1.27)) (justify left bottom))
+  )
   (label "ICSP_MISO" (at 50.8 32.385 180) (fields_autoplaced)
     (effects (font (size 1.27 1.27)) (justify right bottom))
@@
         (path "/894f620e-3404-4a40-a2a7-513bc1d5f99b"
           (reference "C104") (unit 1)
+        )
+      )
+    )
+  )
+  (symbol (lib_id "Switch:SW_Push") (at 271.78 130.175 0) (unit 1)
+    (in_bom yes) (on_board yes) (dnp no) (fields_autoplaced)
+    (property "Reference" "SW101" (at 271.78 121.92 0)
+      (effects (font (size 1.27 1.27)))
+    )
+    (property "Value" "RESET" (at 271.78 124.46 0)
+      (effects (font (size 1.27 1.27)))
+    )
+    (property "Footprint" "Button_Switch_THT:SW_PUSH_6mm_H4.3mm" (at 271.78 125.095 0)
+      (effects (font (size 1.27 1.27)) hide)
+    )
+    (property "Datasheet" "~" (at 271.78 125.095 0)
+      (effects (font (size 1.27 1.27)) hide)
+    )
+    (pin "1")
+    (pin "2")
+    (instances
+      (project "CANIO"
+        (path "/894f620e-3404-4a40-a2a7-513bc1d5f99b"
+          (reference "SW101") (unit 1)
         )
       )
@@
     )
   )
+  (symbol (lib_id "power:GND") (at 280.035 132.08 0) (unit 1)
+    (in_bom yes) (on_board yes) (dnp no)
+    (property "Reference" "#PWR0117" (at 280.035 138.43 0)
+      (effects (font (size 1.27 1.27)) hide)
+    )
+    (property "Value" "GND" (at 280.035 135.89 0)
+      (effects (font (size 1.27 1.27)))
+    )
+    (property "Footprint" "" (at 280.035 132.08 0)
+      (effects (font (size 1.27 1.27)) hide)
+    )
+    (property "Datasheet" "" (at 280.035 132.08 0)
+      (effects (font (size 1.27 1.27)) hide)
+    )
+    (pin "1")
+    (instances
+      (project "CANIO"
+        (path "/894f620e-3404-4a40-a2a7-513bc1d5f99b"
+          (reference "#PWR0117") (unit 1)
+        )
+      )
+    )
+  )
   (symbol (lib_id "Device:R_Small") (at 243.84 37.465 180) (unit 1)
     (in_bom yes) (on_board yes) (dnp no)
@@
         (path "/894f620e-3404-4a40-a2a7-513bc1d5f99b"
           (reference "D101") (unit 1)
+        )
+      )
+    )
+  )
+  (symbol (lib_id "Device:R_Small") (at 173.355 137.795 270) (unit 1)
+    (in_bom yes) (on_board yes) (dnp no)
+    (property "Reference" "R107" (at 173.355 140.335 90)
+      (effects (font (size 1.27 1.27)))
+    )
+    (property "Value" "10K" (at 173.355 142.875 90)
+      (effects (font (size 1.27 1.27)))
+    )
+    (property "Footprint" "Resistor_SMD:R_0805_2012Metric" (at 173.355 137.795 0)
+      (effects (font (size 1.27 1.27)) hide)
+    )
+    (property "Datasheet" "~" (at 173.355 137.795 0)
+      (effects (font (size 1.27 1.27)) hide)
+    )
+    (property "LCSC#" "C269748" (at 173.355 137.795 0)
+      (effects (font (size 1.27 1.27)) hide)
+    )
+    (pin "1")
+    (pin "2")
+    (instances
+      (project "CANIO"
+        (path "/894f620e-3404-4a40-a2a7-513bc1d5f99b"
+          (reference "R107") (unit 1)
         )
       )
@@
         )
       )
+    )
+  )
+  (symbol (lib_id "power:GND") (at 178.435 147.955 0) (unit 1)
+    (in_bom yes) (on_board yes) (dnp no)
+    (property "Reference" "#PWR0116" (at 178.435 154.305 0)
+      (effects (font (size 1.27 1.27)) hide)
+    )
+    (property "Value" "GND" (at 178.435 151.765 0)
+      (effects (font (size 1.27 1.27)))
+    )
+    (property "Footprint" "" (at 178.435 147.955 0)
+      (effects (font (size 1.27 1.27)) hide)
+    )
+    (property "Datasheet" "" (at 178.435 147.955 0)
+      (effects (font (size 1.27 1.27)) hide)
+    )
+    (pin "1")
+    (instances
+      (project "CANIO"
+        (path "/894f620e-3404-4a40-a2a7-513bc1d5f99b"
+          (reference "#PWR0116") (unit 1)
+        )
+      )

Commit message: Design improvements, multilayer and more
Parts:
- added C105: 100nF, Capacitor_SMD:C_0805_2012Metric, symbol Device:C_Small
- added R108: 100R, Resistor_SMD:R_0805_2012Metric, symbol Device:R_Small
Connections:
- net +5V: now also C105.1
- net CLKOUT: now also R108.1; no longer JP101.1 (A)
- net GND: now also C105.2
- new net: JP101.1 (A), R108.2
Changed lines of the file:
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@@
+    (stroke (width 0) (type default))
+  )
+  (wire (pts (xy 101.6 86.995) (xy 104.14 86.995))
     (stroke (width 0) (type default))
   )
@@
     (stroke (width 0) (type default))
   )
+  (wire (pts (xy 179.705 72.39) (xy 179.705 73.66))
+    (stroke (width 0) (type default))
+  )
   (wire (pts (xy 38.1 32.385) (xy 50.8 32.385))
     (stroke (width 0) (type default))
@@
     (stroke (width 0) (type default))
   )
+  (wire (pts (xy 179.705 65.405) (xy 179.705 67.31))
+    (stroke (width 0) (type default))
+  )
   (wire (pts (xy 38.1 34.925) (xy 50.8 34.925))
     (stroke (width 0) (type default))
@@
     (stroke (width 0) (type default))
   )
-  (wire (pts (xy 94.615 86.995) (xy 104.14 86.995))
+  (wire (pts (xy 84.455 86.995) (xy 96.52 86.995))
     (stroke (width 0) (type default))
   )
@@
     (effects (font (size 1.27 1.27)) (justify right bottom))
   )
-  (label "CLKOUT" (at 94.615 86.995 0) (fields_autoplaced)
+  (label "CLKOUT" (at 84.455 86.995 0) (fields_autoplaced)
     (effects (font (size 1.27 1.27)) (justify left bottom))
   )
@@
   )
   (symbol (lib_id "Jumper:SolderJumper_2_Bridged") (at 107.95 86.995 0) (unit 1)
-    (in_bom yes) (on_board yes) (dnp no) (fields_autoplaced)
-    (property "Reference" "JP101" (at 107.95 83.82 0)
+    (in_bom yes) (on_board yes) (dnp no)
+    (property "Reference" "JP101" (at 107.95 90.17 0)
       (effects (font (size 1.27 1.27)))
     )
@@
         (path "/894f620e-3404-4a40-a2a7-513bc1d5f99b"
           (reference "C101") (unit 1)
+        )
+      )
+    )
+  )
+  (symbol (lib_id "power:+5V") (at 179.705 65.405 0) (unit 1)
+    (in_bom yes) (on_board yes) (dnp no)
+    (property "Reference" "#PWR0118" (at 179.705 69.215 0)
+      (effects (font (size 1.27 1.27)) hide)
+    )
+    (property "Value" "+5V" (at 179.705 61.595 0)
+      (effects (font (size 1.27 1.27)))
+    )
+    (property "Footprint" "" (at 179.705 65.405 0)
+      (effects (font (size 1.27 1.27)) hide)
+    )
+    (property "Datasheet" "" (at 179.705 65.405 0)
+      (effects (font (size 1.27 1.27)) hide)
+    )
+    (pin "1")
+    (instances
+      (project "CANIO"
+        (path "/894f620e-3404-4a40-a2a7-513bc1d5f99b"
+          (reference "#PWR0118") (unit 1)
         )
       )
@@
         (path "/894f620e-3404-4a40-a2a7-513bc1d5f99b"
           (reference "#PWR0114") (unit 1)
+        )
+      )
+    )
+  )
+  (symbol (lib_name "GND_5") (lib_id "power:GND") (at 179.705 73.66 0) (unit 1)
+    (in_bom yes) (on_board yes) (dnp no)
+    (property "Reference" "#PWR0119" (at 179.705 80.01 0)
+      (effects (font (size 1.27 1.27)) hide)
+    )
+    (property "Value" "GND" (at 179.705 77.47 0)
+      (effects (font (size 1.27 1.27)))
+    )
+    (property "Footprint" "" (at 179.705 73.66 0)
+      (effects (font (size 1.27 1.27)) hide)
+    )
+    (property "Datasheet" "" (at 179.705 73.66 0)
+      (effects (font (size 1.27 1.27)) hide)
+    )
+    (pin "1")
+    (instances
+      (project "CANIO"
+        (path "/894f620e-3404-4a40-a2a7-513bc1d5f99b"
+          (reference "#PWR0119") (unit 1)
         )
       )
@@
     )
   )
+  (symbol (lib_id "Device:C_Small") (at 179.705 69.85 0) (unit 1)
+    (in_bom yes) (on_board yes) (dnp no)
+    (property "Reference" "C105" (at 184.15 70.485 0)
+      (effects (font (size 1.27 1.27)))
+    )
+    (property "Value" "100nF" (at 184.785 72.39 0)
+      (effects (font (size 1.27 1.27)))
+    )
+    (property "Footprint" "Capacitor_SMD:C_0805_2012Metric" (at 179.705 69.85 0)
+      (effects (font (size 1.27 1.27)) hide)
+    )
+    (property "Datasheet" "~" (at 179.705 69.85 0)
+      (effects (font (size 1.27 1.27)) hide)
+    )
+    (pin "1")
+    (pin "2")
+    (instances
+      (project "CANIO"
+        (path "/894f620e-3404-4a40-a2a7-513bc1d5f99b"
+          (reference "C105") (unit 1)
+        )
+      )
+    )
+  )
   (symbol (lib_id "power:GND") (at 243.84 41.275 0) (unit 1)
     (in_bom yes) (on_board yes) (dnp no)
@@
         )
       )
+    )
+  )
+  (symbol (lib_id "Device:R_Small") (at 99.06 86.995 90) (unit 1)
+    (in_bom yes) (on_board yes) (dnp no)
+    (property "Reference" "R108" (at 99.06 89.535 90)
+      (effects (font (size 1.27 1.27)))
+    )
+    (property "Value" "100R" (at 99.06 91.44 90)
+      (effects (font (size 1.27 1.27)))
+    )
+    (property "Footprint" "Resistor_SMD:R_0805_2012Metric" (at 99.06 86.995 0)
+      (effects (font (size 1.27 1.27)) hide)
+    )
+    (property "Datasheet" "~" (at 99.06 86.995 0)
+      (effects (font (size 1.27 1.27)) hide)
+    )
+    (pin "1")
+    (pin "2")
+    (instances
+      (project "CANIO"
+        (path "/894f620e-3404-4a40-a2a7-513bc1d5f99b"
+          (reference "R108") (unit 1)
+        )
+      )

Commit message: Do some routing
Parts:
- added TP101: STBY, TestPoint:TestPoint_Pad_2.0x2.0mm, symbol Connector:TestPoint
- added TP102, TP103, TP104, TP105, TP106: TestPoint, TestPoint:TestPoint_Pad_2.0x2.0mm, symbol Connector:TestPoint
- P101: LCSC# (none) -> C2765186
Connections:
- net +5V: now also TP106.1
- net ICSP_MISO: now also TP105.1
- net ICSP_MOSI: now also TP104.1
- net ICSP_SCK: now also TP103.1
- net CS: now reaches U101.14 (PB0)
- net CS: now also TP102.1
- net CAN_STBY: now reaches U101.7 (PD1)
- net CAN_STBY: now also TP101.1
- net CAN_INT: now reaches U101.8 (PD2)
- no-connect marks 23 -> 17
Other:
- note added: "If CAN_INT were instead on PC0 We could use a hw inturrupt?"
- note added: "PB0 Can be SS (for the 16u2) or just a general I/O like we're using here."
- note added: "Pull UP to go to standby"
- note removed: "Is standby pullup or down to standby?"

Commit message: Add a few more comments
Other:
- note added: "Only populate these if for some reason the CLKOUT from the MCP chip dosn't pan out!"
Changed lines of the file:
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@@
+    (effects (font (size 1.27 1.27)) (justify left bottom))
+  )
+  (text "Only populate these\nif for some reason the \nCLKOUT from the MCP chip\ndosn't pan out!"
+    (at 81.28 139.7 0)
     (effects (font (size 1.27 1.27)) (justify left bottom))
   )
