File: Hardware/CANIO/canbus.kicad_sch (KiCad schematic)
At the start: 18 parts, among them J201 CAN, J202 CAN, U201 MCP25625-x-SS, Y202 Crystal_GND24

Commit message: Add term solder jumper
Parts:
- added JP201: TERM, Jumper:SolderJumper-2_P1.3mm_Bridged2Bar_Pad1.0x1.5mm, symbol Jumper:SolderJumper_2_Bridged
Connections:
- net CANL: now also JP201.2 (B); no longer R201.1
- new net: JP201.1 (A), R201.1
Changed lines of the file:
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@@
     (stroke (width 0) (type default))
   )
-  (wire (pts (xy 243.84 69.85) (xy 234.95 69.85))
+  (wire (pts (xy 243.84 76.835) (xy 234.95 76.835))
     (stroke (width 0) (type default))
   )
@@
     (stroke (width 0) (type default))
   )
-  (wire (pts (xy 234.95 69.85) (xy 234.95 67.31))
+  (wire (pts (xy 234.95 76.835) (xy 234.95 75.565))
+    (stroke (width 0) (type default))
+  )
+  (wire (pts (xy 234.95 67.945) (xy 234.95 67.31))
     (stroke (width 0) (type default))
   )
@@
     (effects (font (size 1.27 1.27)) (justify left bottom))
   )
-  (label "CANL" (at 243.84 69.85 180) (fields_autoplaced)
+  (label "CANL" (at 243.84 76.835 180) (fields_autoplaced)
     (effects (font (size 1.27 1.27)) (justify right bottom))
   )
@@
         )
       )
+    )
+  )
+  (symbol (lib_id "Jumper:SolderJumper_2_Bridged") (at 234.95 71.755 270) (unit 1)
+    (in_bom yes) (on_board yes) (dnp no)
+    (property "Reference" "JP201" (at 231.775 71.755 0)
+      (effects (font (size 1.27 1.27)))
+    )
+    (property "Value" "TERM" (at 238.125 71.755 0)
+      (effects (font (size 1.27 1.27)) hide)
+    )
+    (property "Footprint" "Jumper:SolderJumper-2_P1.3mm_Bridged2Bar_Pad1.0x1.5mm" (at 234.95 71.755 0)
+      (effects (font (size 1.27 1.27)) hide)
+    )
+    (property "Datasheet" "~" (at 234.95 71.755 0)
+      (effects (font (size 1.27 1.27)) hide)
+    )
+    (pin "2")
+    (pin "1")
+    (instances
+      (project "CANIO"
+        (path "/894f620e-3404-4a40-a2a7-513bc1d5f99b/de3f136a-4876-4908-a268-32055f46152a"
+          (reference "JP201") (unit 1)
+        )
+      )
